Commit message: tof 3d

File: nexen_bot/description/gazebo_control.xacro (robot description, xacro)
@@ -6,6 +6,6 @@
             <left_joint>left_wheel_joint</left_joint>
             <right_joint>right_wheel_joint</right_joint>
-            <wheel_separation>0.297</wheel_separation>
-            <wheel_diameter>0.066</wheel_diameter>
+            <wheel_separation>0.345</wheel_separation>
+            <wheel_diameter>0.088</wheel_diameter>
             <!-- Limits -->
             <max_wheel_torque>200</max_wheel_torque>

File: nexen_bot/description/robot_core.xacro (robot description, xacro)
@@ -67,5 +67,5 @@
     </link>
     <gazebo reference="chassis">
-        <material>Gazebo/Orange</material>
+        <material>Gazebo/White</material>
     </gazebo>
     <!-- LEFT WHEEL LINK -->

File: nexen_bot/description/ros2_control.xacro (robot description, xacro)
@@ -11,5 +11,5 @@
                 <param name="baud_rate">57600</param>
                 <param name="timeout">1000</param>
-                <param name="enc_counts_per_rev">1000</param>
+                <param name="enc_counts_per_rev">1008</param>
             </hardware>
             <joint name="left_wheel_joint">

Commit message: white colour

File: nexen_bot/description/gazebo_control.xacro (robot description, xacro)
@@ -6,6 +6,6 @@
             <left_joint>left_wheel_joint</left_joint>
             <right_joint>right_wheel_joint</right_joint>
-            <wheel_separation>0.345</wheel_separation>
-            <wheel_diameter>0.088</wheel_diameter>
+            <wheel_separation>0.35</wheel_separation>
+            <wheel_diameter>0.090</wheel_diameter>
             <!-- Limits -->
             <max_wheel_torque>200</max_wheel_torque>

File: nexen_bot/description/robot_core.xacro (robot description, xacro)
@@ -2,15 +2,15 @@
 <robot xmlns:xacro="http://www.ros.org/wiki/xacro" >
     <xacro:include filename="inertial_macros.xacro"/>
-    <xacro:property name="chassis_length" value="0.385"/>
+    <xacro:property name="chassis_length" value="0.389"/>
     <xacro:property name="chassis_width" value="0.305"/>
     <xacro:property name="chassis_height" value="0.24"/>
     <xacro:property name="chassis_mass" value="1.0"/>
-    <xacro:property name="wheel_radius" value="0.044"/>
-    <xacro:property name="wheel_thickness" value="0.008"/>
+    <xacro:property name="wheel_radius" value="0.045"/>
+    <xacro:property name="wheel_thickness" value="0.01"/>
     <xacro:property name="wheel_mass" value="0.05"/>
-    <xacro:property name="wheel_offset_x" value="0.29"/>
-    <xacro:property name="wheel_offset_y" value="0.1725"/>
-    <xacro:property name="wheel_offset_z" value="-0.0175"/>
-    <xacro:property name="caster_wheel_radius" value="0.01"/>
+    <xacro:property name="wheel_offset_x" value="0.30"/>
+    <xacro:property name="wheel_offset_y" value="0.175"/>
+    <xacro:property name="wheel_offset_z" value="0.01"/>
+    <xacro:property name="caster_wheel_radius" value="0.12"/>
     <xacro:property name="caster_wheel_mass" value="0.01"/>
     <xacro:property name="caster_wheel_offset_x" value="0.01"/>
